Commit message: sync

File: simulation/models/jag.urdf (robot description, URDF)
Before this commit: robot jaguar, 18 links, 17 joints
Joints:
- joint camera_joint: origin xyz=0.24 0 0.315 rpy=0 0.2 0 -> xyz=0.3 0 0.19 rpy=0 0.2 0

Commit message: change in orientation to goal

File: simulation/models/jag.urdf (robot description, URDF)
Before this commit: robot jaguar, 18 links, 17 joints
Links:
- link arm_1: geometry visual mesh filename=package://simulation/models/meshes/jaguar/arm1.dae scale=0.021 0.021 0.021
- link arm_2: geometry visual mesh filename=package://simulation/models/meshes/jaguar/arm2.dae scale=0.021 0.021 0.021
- link arm_3: geometry visual mesh filename=package://simulation/models/meshes/jaguar/arm3.dae scale=0.021 0.021 0.021

Commit message: flat world representation changed

File: simulation/models/jag.urdf (robot description, URDF)
Before this commit: robot jaguar, 18 links, 17 joints
Joints:
- joint camera_joint: origin xyz=0.3 0 0.19 rpy=0 0.2 0 -> xyz=0.3 0 0.19 rpy=0 0.0 0

Commit message: string to bool check

File: simulation/models/jag.urdf (robot description, URDF)
Before this commit: robot jaguar, 18 links, 17 joints
Joints:
- joint camera_joint: origin xyz=0.3 0 0.19 rpy=0 0.0 0 -> xyz=0.175 0.1 0.355 rpy=0 0.47 0.0

Commit message: sr300 camera integration

File: simulation/models/jag.urdf (robot description, URDF)
Before this commit: robot jaguar, 18 links, 17 joints
Joints:
- joint camera_joint: origin xyz=0.175 0.1 0.355 rpy=0 0.47 0.0 -> xyz=0.21 0.1 0.28 rpy=0 0.43 0.0

Commit message: control improved

File: simulation/models/jag.urdf (robot description, URDF)
Before this commit: robot jaguar, 18 links, 17 joints
Joints:
- joint camera_joint: origin xyz=0.21 0.1 0.28 rpy=0 0.43 0.0 -> xyz=0.195 0.1 0.295 rpy=0 0.46 0.0
